File: USB_Fan.kicad_sch (KiCad schematic)
At the start: 41 parts, among them J1 USB-C (Female), J2 Fan, J3 Fan Voltage, SW1 Power, U1 TP4056, U2 DW01A-G, U3 FS8205A, U4 TPS61170

Commit message: Fix problems on the PCB
Parts:
- removed C6: 1uF, Capacitor_SMD:C_0603_1608Metric, symbol Device:C_Small
- removed L2: 10uH, Custom:Inductor 4x4, symbol Device:L_Small
- R7: footprint Resistor_SMD:R_0805_2012Metric -> Resistor_SMD:R_0603_1608Metric
- renumbered C7 to C6
Connections:
- net at D1.2 (A): now also L1.2, U4.4 (SW)
Other:
- title: TP4056 Charger -> USB Fan
Changed lines of the file:
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@@
   (paper "A4")
   (title_block
-    (title "TP4056 Charger")
+    (title "USB Fan")
     (company "Abit Gray")
   )
@@
   )
   (junction (at 233.68 34.29) (diameter 0) (color 0 0 0 0)
-  )
-  (junction (at 241.3 34.29) (diameter 0) (color 0 0 0 0)
   )
   (junction (at 93.98 66.04) (diameter 0) (color 0 0 0 0)
@@
     (stroke (width 0) (type default))
   )
-  (wire (pts (xy 241.3 36.83) (xy 241.3 34.29))
-    (stroke (width 0) (type default))
-  )
   (wire (pts (xy 270.51 50.8) (xy 270.51 53.34))
     (stroke (width 0) (type default))
@@
     (stroke (width 0) (type default))
   )
-  (wire (pts (xy 233.68 34.29) (xy 236.22 34.29))
+  (wire (pts (xy 233.68 34.29) (xy 241.3 34.29))
     (stroke (width 0) (type default))
   )
@@
   (symbol (lib_id "Device:C_Small") (at 246.38 64.77 0) (mirror y) (unit 1)
     (in_bom yes) (on_board yes) (dnp no)
-    (property "Reference" "C7" (at 243.84 63.5063 0)
+    (property "Reference" "C6" (at 243.84 63.5063 0)
       (effects (font (size 1.27 1.27)) (justify left))
     )
@@
       (project "USB_Fan"
         (path "/16a89f0a-88d3-42f5-a8f1-2ef510493fd4"
-          (reference "C7") (unit 1)
+          (reference "C6") (unit 1)
         )
       )
@@
     )
   )
-  (symbol (lib_id "Device:L_Small") (at 241.3 39.37 180) (unit 1)
-    (in_bom yes) (on_board yes) (dnp no)
-    (property "Reference" "L2" (at 242.57 38.1 0)
-      (effects (font (size 1.27 1.27)) (justify right))
-    )
-    (property "Value" "10uH" (at 242.57 40.64 0)
-      (effects (font (size 1.27 1.27)) (justify right))
-    )
-    (property "Footprint" "Custom:Inductor 4x4" (at 241.3 39.37 0)
-      (effects (font (size 1.27 1.27)) hide)
-    )
-    (property "Datasheet" "~" (at 241.3 39.37 0)
-      (effects (font (size 1.27 1.27)) hide)
-    )
-    (property "LCSC" "C497803" (at 241.3 39.37 0)
-      (effects (font (size 1.27 1.27)) hide)
-    )
-    (pin "1")
-    (pin "2")
-    (instances
-      (project "USB_Fan"
-        (path "/16a89f0a-88d3-42f5-a8f1-2ef510493fd4"
-          (reference "L2") (unit 1)
-        )
-      )
-    )
-  )
   (symbol (lib_id "power:GND") (at 196.85 57.15 0) (unit 1)
     (in_bom yes) (on_board yes) (dnp no)
@@
         (path "/16a89f0a-88d3-42f5-a8f1-2ef510493fd4"
           (reference "#PWR0114") (unit 1)
-        )
-      )
-    )
-  )
-  (symbol (lib_id "power:GND") (at 241.3 41.91 0) (unit 1)
-    (in_bom yes) (on_board yes) (dnp no)
-    (property "Reference" "#PWR0111" (at 241.3 48.26 0)
-      (effects (font (size 1.27 1.27)) hide)
-    )
-    (property "Value" "GND" (at 241.3 45.72 0)
-      (effects (font (size 1.27 1.27)))
-    )
-    (property "Footprint" "" (at 241.3 41.91 0)
-      (effects (font (size 1.27 1.27)) hide)
-    )
-    (property "Datasheet" "" (at 241.3 41.91 0)
-      (effects (font (size 1.27 1.27)) hide)
-    )
-    (pin "1")
-    (instances
-      (project "USB_Fan"
-        (path "/16a89f0a-88d3-42f5-a8f1-2ef510493fd4"
-          (reference "#PWR0111") (unit 1)
         )
       )
@@
       (effects (font (size 1.27 1.27)))
     )
-    (property "Footprint" "Resistor_SMD:R_0805_2012Metric" (at 166.37 31.242 90)
+    (property "Footprint" "Resistor_SMD:R_0603_1608Metric" (at 166.37 31.242 90)
       (effects (font (size 1.27 1.27)) hide)
     )
@@
         )
       )
-    )
-  )
-  (symbol (lib_id "Device:C_Small") (at 238.76 34.29 90) (mirror x) (unit 1)
-    (in_bom yes) (on_board yes) (dnp no)
-    (property "Reference" "C6" (at 238.76 31.75 90)
-      (effects (font (size 1.27 1.27)))
-    )
-    (property "Value" "1uF" (at 238.76 36.83 90)
-      (effects (font (size 1.27 1.27)))
-    )
-    (property "Footprint" "Capacitor_SMD:C_0603_1608Metric" (at 238.76 34.29 0)
-      (effects (font (size 1.27 1.27)) hide)
-    )
-    (property "Datasheet" "~" (at 238.76 34.29 0)
-      (effects (font (size 1.27 1.27)) hide)
-    )
-    (property "LCSC" "C15849" (at 238.76 34.29 0)
-      (effects (font (size 1.27 1.27)) hide)
-    )
-    (pin "1")
-    (pin "2")
-    (instances
-      (project "USB_Fan"
-        (path "/16a89f0a-88d3-42f5-a8f1-2ef510493fd4"
-          (reference "C6") (unit 1)
-        )
-      )

Commit message: Add tooling holes
Parts:
- H1, H2: footprint Custom:Tooling Hole (JLCPCB) -> Custom:JLCPCB ToolingHole
Changed lines of the file:
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@@
       (effects (font (size 1.27 1.27)) (justify left) hide)
     )
-    (property "Footprint" "Custom:Tooling Hole (JLCPCB)" (at 242.57 147.32 0)
+    (property "Footprint" "Custom:JLCPCB ToolingHole" (at 242.57 147.32 0)
       (effects (font (size 1.27 1.27)) hide)
     )
     (property "Datasheet" "~" (at 242.57 147.32 0)
+      (effects (font (size 1.27 1.27)) hide)
+    )
+    (property "LCSC" "" (at 242.57 147.32 0)
       (effects (font (size 1.27 1.27)) hide)
     )
@@
       (effects (font (size 1.27 1.27)) (justify left) hide)
     )
-    (property "Footprint" "Custom:Tooling Hole (JLCPCB)" (at 248.92 147.32 0)
+    (property "Footprint" "Custom:JLCPCB ToolingHole" (at 248.92 147.32 0)
       (effects (font (size 1.27 1.27)) hide)
     )
@@
       (effects (font (size 1.27 1.27)) hide)
     )
+    (property "LCSC" "" (at 248.92 147.32 0)
+      (effects (font (size 1.27 1.27)) hide)
+    )
