File: USB_Fan.kicad_sch (KiCad schematic)
At the start: 39 parts, among them J1 USB-C (Female), J2 Fan, J3 Fan Voltage, SW1 Power, U1 TP4056, U2 DW01A-G, U3 FS8205A, U4 TPS61170

Commit message: Revision 2
Parts:
- H1, H2, H3, H4, H5, H6, J3, SW1: LCSC (none) -> -
Connections:
- net -BATT: now also U3.1 (S1); no longer U3.3 (S2)
- net FET Charge: now also U3.4 (G2); no longer U3.6 (G1)
- net FET Discharge: now also U3.6 (G1); no longer U3.4 (G2)
- net GND: now also J1.S1 (SHIELD), U3.3 (S2); no longer U3.1 (S1)
- no-connect marks 10 -> 9
Other:
- moved on the sheet: J1, R1, R2

Commit message: Minor tweak for manufacturing
Parts:
- BT1: LCSC (none) -> C18077744
- D3: LCSC (none) -> C965827
- D4: LCSC (none) -> C2827254
- J2: LCSC (none) -> C234181
Changed lines of the file:
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@@
 			)
 		)
-		(property "LCSC" ""
+		(property "LCSC" "C18077744"
 			(at 177.8 40.64 0)
 			(effects
@@
 			)
 		)
+		(property "LCSC" "C965827"
+			(at 68.58 38.1 0)
+			(effects
+				(font
+					(size 1.27 1.27)
+				)
+				(hide yes)
+			)
+		)
 		(pin "1"
 		)
@@
 			)
 		)
+		(property "LCSC" "C2827254"
+			(at 76.2 38.1 0)
+			(effects
+				(font
+					(size 1.27 1.27)
+				)
+				(hide yes)
+			)
+		)
 		(pin "1"
 		)
@@
 			)
 		)
-		(property "LCSC" ""
+		(property "LCSC" "C234181"
 			(at 252.73 69.85 0)
 			(effects
